Commit message: fixed chassis urdf error

File: urdf/rabbit/chassis.urdf.xacro (robot description, xacro)
@@ -2,5 +2,5 @@
     <xacro:include filename="$(find rc_description)/urdf/common/mecanum_wheel.urdf.xacro"/>
     <xacro:property name="wheel_track" value="0.37116"/>
-    <xacro:property name="wheel_base" value="0.4164"/>
+    <xacro:property name="wheel_base" value="0.4664"/>
     <xacro:property name="wheel_offset_z" value="-0.02"/>
     <xacro:macro name="chassis" params="roller_type">

File: urdf/rabbit/rabbit.urdf.xacro (robot description, xacro)
@@ -9,6 +9,6 @@
     <xacro:arg name="load_collect" default="false"/>
     <xacro:arg name="load_collect_transmission" default="false"/>
-    <xacro:arg name="load_radar" default="false"/>
-    <xacro:arg name="load_action" default="false"/>
+    <xacro:arg name="load_radar" default="true"/>
+    <xacro:arg name="load_action" default="true"/>
     <xacro:arg name="use_sim" default="true"/>
     <xacro:arg name="use_simulation" default="false"/>
